File: kicad/3APSU.kicad_sch (KiCad schematic)
At the start: 53 parts, among them P1 9VAC, P10 -12V, P2 9VAC, P3 15VAC, P4 GND, P5 15VAC, P6 +5V, P7 0V, P8 +12V, P9 -5V, U1 LM323K, U2 L7812, U3 L7905, U4 L7912

Commit message: Kicad 9 update
Other:
- title: 3A PSU -> 3A PSU / Kicad 9
